Commit message: Demo specific changes

File: panda_moveit_config/srdf/panda_arm.xacro (robot description, xacro)
@@ -19,4 +19,22 @@
       <joint name="${prefix}joint6" value="${pi/2}"/>
       <joint name="${prefix}joint7" value="${pi/4}"/>
+    </group_state>
+    <group_state group="arm" name="start">
+      <joint name="${prefix}joint1" value="0.0"/>
+      <joint name="${prefix}joint2" value="-0.690"/>
+      <joint name="${prefix}joint3" value="0.0"/>
+      <joint name="${prefix}joint4" value="-2.905"/>
+      <joint name="${prefix}joint5" value="0.0"/>
+      <joint name="${prefix}joint6" value="2.2145"/>
+      <joint name="${prefix}joint7" value="0.7852"/>
+    </group_state>
+    <group_state group="arm" name="goal">
+      <joint name="${prefix}joint1" value="-1.10516"/>
+      <joint name="${prefix}joint2" value="-0.61752"/>
+      <joint name="${prefix}joint3" value="1.41199"/>
+      <joint name="${prefix}joint4" value="-2.9175"/>
+      <joint name="${prefix}joint5" value="1.12897"/>
+      <joint name="${prefix}joint6" value="2.45685"/>
+      <joint name="${prefix}joint7" value="0.01927"/>
     </group_state>
     <group_state group="arm" name="extended">
